Commit message: shoulder and wrist

File: hw2/urdf/test.urdf (robot description, URDF)
Before this commit: robot materials, 4 links, 3 joints
Links:
- added link left_wrist; visual box size=0.01 0.01 0.2
Joints:
- added joint left_wrist_joint: type revolute, parent left_shoulder, child left_wrist, origin xyz=0.0 0. 0.2 rpy=0.0 0.0 0.0, axis 0 1 0, limit lower=-1.570795 upper=1.570795 effort=30 velocity=1.0
